Commit message: add worlds and basic gazebo launch file
Signed-off-by: Kenji Brameld <kenjibrameld@gmail.com>

File: urdf/bot.urdf (robot description, URDF)
Before this commit: robot bot, 2 links, 1 joints
Links:
- added link world
Joints:
- added joint base: type fixed, parent world, child link1

Commit message: add second joint
Signed-off-by: Kenji Brameld <kenjibrameld@gmail.com>

File: urdf/bot.urdf (robot description, URDF)
Before this commit: robot bot, 3 links, 2 joints
Links:
- added link link3, mass 0.2; visual box size=0.05 0.05 0.50
Joints:
- added joint joint2: type revolute, parent link2, child link3, origin xyz=0.0 0.0 0.5, axis 1.0 0.0 0.0, limit lower=-1.0 upper=1.0 effort=10.0 velocity=10.0
